Commit message: Changing urdf model

File: urdfbot_description/urdf/urdfbot_simple.urdf (robot description, URDF)
Before this commit: robot urdfbot, 1 links, 0 joints
Links:
- added link head_link; visual box size=0.1 0.1 0.1
Joints:
- added joint base_link_to_head_link_joint: type fixed, parent base_link, child head_link, origin xyz=0 0 0.11 rpy=0 0 0
